File: pcb/ukiha-draft.kicad_pcb (KiCad board)
At the start: 2 copper layers, 326.5 x 241.5 mm, 76 parts, among them SW10 SW_Push, SW11 SW_Push, SW12 SW_Push, SW20 SW_Push, SW21 SW_Push, SW22 SW_Push, SW23 SW_Push, SW24 SW_Push, SW32 SW_Push, SW33 SW_Push, SW34 SW_Push, SW35 SW_Push, SW36 SW_Push, SW44 SW_Push, SW45 SW_Push, SW46 SW_Push, SW47 SW_Push, SW48 SW_Push, SW56 SW_Push, SW57 SW_Push, SW58 SW_Push, SW59 SW_Push, SW60 SW_Push, SW8 SW_Push, SW9 SW_Push

Commit message: Add 48 key middle plate
Parts:
- removed the ? at (29.1, 235.8)
- removed the ? at (-96.9, 158.3)
- removed the ? at (95.1, 190.3)
- removed the ? at (29.1, 174.3)
- removed the ? at (29.1, 190.3)
- removed the ? at (95.1, 38.8)
- removed the ? at (159.1, 38.8)
- removed the ? at (225.1, 38.8)
- removed the ? at (225.1, 54.8)
- removed the ? at (225.1, 106.8)
- removed the ? at (225.1, 122.8)
- removed the ? at (29.1, 219.8)
- removed the ? at (159.1, 122.8)
- removed the ? at (95.1, 122.8)
- removed the ? at (29.1, 122.8)
- removed the ? at (29.1, 106.8)
- removed the ? at (29.1, 54.8)
- removed the ? at (29.1, 38.8)
- removed the ? at (95.1, 235.8)
- removed the ? at (-96.9, 217.8)
- removed the ? at (-30.9, 217.8)
- removed the ? at (-97.4, 67.3)
- removed the ? at (-31.4, 67.3)
- removed the ? at (-96.9, 142.3)
- removed the ? at (-30.9, 142.3)
- added ?: , #footprint:M2_Hole, F.Cu at (159.1, 54.8)
- added ?: , #footprint:M2_Hole, F.Cu at (225.1, 106.8)
- added ?: , #footprint:M2_Hole, F.Cu at (29.1, 106.8)
- added ?: , #footprint:M2_Hole, F.Cu at (29.1, 122.8)
- added ?: , #footprint:M2_Hole, F.Cu at (29.1, 54.8)
- added ?: , #footprint:M2_Hole, F.Cu at (29.1, 38.8)
- added ?: , #footprint:M2_Hole, F.Cu at (95.1, 54.8)
- added ?: , #footprint:M2_Hole, F.Cu at (95.1, 122.8)
- added ?: , #footprint:M2_Hole, F.Cu at (159.1, 122.8)
- added ?: , #footprint:M2_Hole, F.Cu at (159.1, 38.8)
- added ?: , #footprint:M2_Hole, F.Cu at (95.1, 38.8)
- added ?: , #footprint:M2_Hole, F.Cu at (225.1, 38.8)
- added ?: , #footprint:M2_Hole, F.Cu at (225.1, 54.8)
- added ?: , #footprint:M2_Hole, F.Cu at (225.1, 122.8)
- added D1: D, #footprint:diode_SMD, F.Cu at (35.9, 42.8)
- added D13: D, #footprint:diode_SMD, F.Cu at (43.1, 68.8)
- added D14: D, #footprint:diode_SMD, F.Cu at (59.1, 68.8)
- added D15: D, #footprint:diode_SMD, F.Cu at (71.1, 69.8)
- added D16: D, #footprint:diode_SMD, F.Cu at (87.1, 69.8)
- added D17: D, #footprint:diode_SMD, F.Cu at (103.1, 69.8)
- added D18: D, #footprint:diode_SMD, F.Cu at (119.1, 69.8)
- added D19: D, #footprint:diode_SMD, F.Cu at (135.1, 69.8)
- added D2: D, #footprint:diode_SMD, F.Cu at (51.9, 42.8)
- added D25: D, #footprint:diode_SMD, F.Cu at (35.1, 68.8)
- added D26: D, #footprint:diode_SMD, F.Cu at (51.1, 68.8)
- added D27: D, #footprint:diode_SMD, F.Cu at (71.1, 85.8)
- added D28: D, #footprint:diode_SMD, F.Cu at (87.1, 85.8)
- added D29: D, #footprint:diode_SMD, F.Cu at (103.1, 85.8)
- added D3: D, #footprint:diode_SMD, F.Cu at (67.9, 42.8)
- added D30: D, #footprint:diode_SMD, F.Cu at (119.1, 85.8)
- added D31: D, #footprint:diode_SMD, F.Cu at (135.1, 85.8)
- added D37: D, #footprint:diode_SMD, F.Cu at (35.6, 92.3)
- added D38: D, #footprint:diode_SMD, F.Cu at (51.9, 92.3)
- added D39: D, #footprint:diode_SMD, F.Cu at (67.9, 90.8)
- added D4: D, #footprint:diode_SMD, F.Cu at (83.9, 42.8)
- added D40: D, #footprint:diode_SMD, F.Cu at (83.9, 90.8)
- added D41: D, #footprint:diode_SMD, F.Cu at (99.9, 90.8)
- added D42: D, #footprint:diode_SMD, F.Cu at (115.9, 90.8)
- added D43: D, #footprint:diode_SMD, F.Cu at (131.9, 90.8)
- added D49: D, #footprint:diode_SMD, F.Cu at (39.1, 117.8)
- added D5: D, #footprint:diode_SMD, F.Cu at (99.9, 42.8)
- added D50: D, #footprint:diode_SMD, F.Cu at (55.1, 117.8)
- added D51: D, #footprint:diode_SMD, F.Cu at (71.1, 117.8)
- added D52: D, #footprint:diode_SMD, F.Cu at (87.1, 117.8)
- added D53: D, #footprint:diode_SMD, F.Cu at (103.1, 117.8)
- added D54: D, #footprint:diode_SMD, F.Cu at (119.1, 117.8)
- added D55: D, #footprint:diode_SMD, F.Cu at (135.1, 117.8)
- added D6: D, #footprint:diode_SMD, F.Cu at (115.1, 42.8)
- added D61: D, #footprint:diode_SMD, F.Cu at (111.1, 117.8)
- added D63: D, #footprint:diode_SMD, F.Cu at (127.1, 117.8)
- added D7: D, #footprint:diode_SMD, F.Cu at (131.9, 42.8)
- added G***: LOGO, #footprint:e3w2q_icon, B.Cu at (32.6, 121.1)
- added J1: Conn_01x03, #footprint:StripLED_rev2, F.Cu at (39.1, 105.5)
- added SW1: SW_Push, #footprint:CherryMX_MidHeight_16mm_rev2, F.Cu at (39.1, 48.8)
- added SW13: SW_Push, #footprint:CherryMX_MidHeight_16mm_rev2, F.Cu at (39.1, 64.8)
- added SW14: SW_Push, #footprint:CherryMX_MidHeight_16mm_rev2, F.Cu at (55.1, 64.8)
- added SW15: SW_Push, #footprint:CherryMX_MidHeight_16mm_rev2, F.Cu at (71.1, 64.8)
- added SW16: SW_Push, #footprint:CherryMX_MidHeight_16mm_rev2, F.Cu at (87.1, 64.8)
- added SW17: SW_Push, #footprint:CherryMX_MidHeight_16mm_rev2, F.Cu at (103.1, 64.8)
- added SW18: SW_Push, #footprint:CherryMX_MidHeight_16mm_rev2, F.Cu at (119.1, 64.8)
- added SW19: SW_Push, #footprint:CherryMX_MidHeight_16mm_rev2, F.Cu at (135.1, 64.8)
- added SW2: SW_Push, #footprint:CherryMX_MidHeight_16mm_rev2, F.Cu at (55.1, 48.8)
- added SW25: SW_Push, #footprint:CherryMX_MidHeight_16mm_rev2, F.Cu at (39.1, 80.8)
- added SW26: SW_Push, #footprint:CherryMX_MidHeight_16mm_rev2, F.Cu at (55.1, 80.8)
- added SW27: SW_Push, #footprint:CherryMX_MidHeight_16mm_rev2, F.Cu at (71.1, 80.8)
- added SW28: SW_Push, #footprint:CherryMX_MidHeight_16mm_rev2, F.Cu at (87.1, 80.9)
- added SW29: SW_Push, #footprint:CherryMX_MidHeight_16mm_rev2, F.Cu at (103.1, 80.8)
- added SW3: SW_Push, #footprint:CherryMX_MidHeight_16mm_rev2, F.Cu at (71.1, 48.8)
- added SW30: SW_Push, #footprint:CherryMX_MidHeight_16mm_rev2, F.Cu at (119.1, 80.8)
- added SW31: SW_Push, #footprint:CherryMX_MidHeight_16mm_rev2, F.Cu at (135.1, 80.8)
- added SW37: SW_Push, #footprint:CherryMX_MidHeight_16mm_rev2, F.Cu at (39.1, 96.8)
- added SW38: SW_Push, #footprint:CherryMX_MidHeight_16mm_rev2, F.Cu at (55.1, 96.8)
- added SW39: SW_Push, #footprint:CherryMX_MidHeight_16mm_rev2, F.Cu at (71.1, 96.8)
- added SW4: SW_Push, #footprint:CherryMX_MidHeight_16mm_rev2, F.Cu at (87.1, 48.8)
- added SW40: SW_Push, #footprint:CherryMX_MidHeight_16mm_rev2, F.Cu at (87.1, 96.8)
- added SW41: SW_Push, #footprint:CherryMX_MidHeight_16mm_rev2, F.Cu at (103.1, 96.8)
- added SW42: SW_Push, #footprint:CherryMX_MidHeight_16mm_rev2, F.Cu at (119.1, 96.8)
- added SW43: SW_Push, #footprint:CherryMX_MidHeight_16mm_rev2, F.Cu at (135.1, 96.8)
- added SW49: SW_Push, #footprint:CherryMX_MidHeight_16mm_rev2, F.Cu at (39.1, 112.8)
- added SW5: SW_Push, #footprint:CherryMX_MidHeight_16mm_rev2, F.Cu at (103.1, 48.8)
- added SW50: SW_Push, #footprint:CherryMX_MidHeight_16mm_rev2, F.Cu at (55.1, 112.8)
- added SW51: SW_Push, #footprint:CherryMX_MidHeight_16mm_rev2, F.Cu at (71.1, 112.8)
- added SW52: SW_Push, #footprint:CherryMX_MidHeight_16mm_rev2, F.Cu at (87.1, 112.8)
- added SW53: SW_Push, #footprint:CherryMX_MidHeight_16mm_rev3, F.Cu at (103.1, 112.8)
- added SW54: SW_Push, #footprint:CherryMX_MidHeight_16mm_rev3, F.Cu at (119.1, 112.8)
- added SW55: SW_Push, #footprint:CherryMX_MidHeight_16mm_rev3, F.Cu at (135.1, 112.8)
- added SW6: SW_Push, #footprint:CherryMX_MidHeight_16mm_rev2, F.Cu at (119.1, 48.8)
- added SW61: SW_Push, #footprint:CherryMX_MidHeight_16mm_rev3, F.Cu at (111.1, 112.8)
- added SW62: SW_Push, #footprint:CherryMX_MidHeight_16mm_rev3, F.Cu at (143.1, 112.8)
- added SW63: SW_Push, #footprint:CherryMX_MidHeight_16mm_rev3, F.Cu at (127.1, 112.8)
- added SW7: SW_Push, #footprint:CherryMX_MidHeight_16mm_rev2, F.Cu at (135.1, 48.8)
- added U1: ProMicro/BLEMicroPro, #footprint:ArduinoProMicro_ConThrough, B.Cu at (46.1, 80.8)
- SW56, SW57, SW58, SW59, SW60: footprint #footprint:CherryMX_MidHeight_16mm_rev2 -> #footprint:CherryMX_MidHeight_16mm_rev3
- moved D47 1.25 mm to (195.9, 90.8)
- moved D48 1.25 mm to (211.9, 90.8)
- moved D23 1.00 mm to (199.1, 69.8)
- moved D24 1.00 mm to (215.1, 69.8)
- moved D10 0.75 mm to (179.9, 42.8)
- moved D11 0.75 mm to (195.9, 42.8)
- moved D12 0.75 mm to (211.9, 42.8)
- moved D44 0.75 mm to (147.9, 90.8)
- moved D45 0.75 mm to (163.9, 90.8)
- moved D46 0.75 mm to (179.9, 90.8)
- moved D8 0.75 mm to (147.9, 42.8)
- moved D9 0.75 mm to (163.9, 42.8)
Routing:
- net Y1: track 0.00 -> 247.8 mm
- net Y3: track 0.00 -> 238.9 mm, vias 0 -> 3
- net X12: track 0.00 -> 229.9 mm
- net Y5: track 0.00 -> 216.7 mm, vias 0 -> 1
- net X11: track 0.00 -> 213.0 mm, vias 0 -> 1
- net Y2: track 0.00 -> 201.9 mm, vias 0 -> 1
- net X10: track 0.00 -> 198.0 mm
- net Y4: track 0.00 -> 191.6 mm, vias 0 -> 2
- net X9: track 0.00 -> 184.1 mm
- net X8: track 0.00 -> 171.2 mm, vias 0 -> 2
- net X7: track 0.00 -> 166.1 mm, vias 0 -> 2
- net X6: track 0.00 -> 152.8 mm
- net X5: track 0.00 -> 141.7 mm
- net X1: track 0.00 -> 105.8 mm, vias 0 -> 1
- net X4: track 0.00 -> 95.7 mm, vias 0 -> 1
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Other:
- board size 326.5 x 241.5 mm -> 200 x 88 mm
- board text added: "Ukiha by @e3w2q"
