File: pcb/ukiha-bottom.kicad_pcb (KiCad board)
At the start: 2 copper layers, 200 x 88 mm, 15 parts

Commit message: Fix PCB
Other:
- outline, holes or cut-outs redrawn
Changed lines of the file:
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@@
   (general
     (thickness 1.6)
-    (drawings 66)
+    (drawings 67)
     (tracks 0)
     (zones 0)
@@
     (pad_to_mask_clearance 0.2)
     (solder_mask_min_width 0.25)
-    (aux_axis_origin 37.70322 52.784508)
+    (aux_axis_origin 27.102501 36.80625)
     (grid_origin 27.102501 36.80625)
     (visible_elements 7FFFFFEF)
@@
       (xy -30.405765 -9.332446) (xy -30.382289 -9.328992) (xy -30.351154 -9.327826) (xy -30.308212 -9.328787)) (layer B.Mask) (width 0.01))
   )
+  (gr_line (start 27.602501 90.80625) (end 62.102501 90.80625) (layer F.Fab) (width 0.15))
   (gr_line (start 127.102501 52.80625) (end 127.102501 66.80625) (layer F.Fab) (width 0.15))
   (gr_line (start 127.102501 110.80625) (end 127.102501 124.80625) (layer F.Fab) (width 0.15))
@@
   (gr_line (start 95.102501 54.80625) (end 159.102501 122.80625) (layer F.Fab) (width 0.15))
   (gr_arc (start 27.602501 70.30625) (end 27.102501 70.30625) (angle -90) (layer Edge.Cuts) (width 0.15))
-  (gr_arc (start 27.602501 91.30625) (end 27.602501 90.80625) (angle -90) (layer Edge.Cuts) (width 0.15))
-  (gr_line (start 27.102501 91.30625) (end 27.102501 122.80625) (layer Edge.Cuts) (width 0.15))
-  (gr_line (start 62.102501 90.80625) (end 27.602501 90.80625) (layer Edge.Cuts) (width 0.15))
-  (gr_line (start 62.102501 70.80625) (end 62.102501 90.80625) (layer Edge.Cuts) (width 0.15))
+  (gr_arc (start 27.602501 90.80625) (end 27.602501 90.30625) (angle -90) (layer Edge.Cuts) (width 0.15))
+  (gr_line (start 27.102501 90.80625) (end 27.102501 122.80625) (layer Edge.Cuts) (width 0.15))
+  (gr_line (start 62.102501 90.30625) (end 27.602501 90.30625) (layer Edge.Cuts) (width 0.15))
+  (gr_line (start 62.102501 70.80625) (end 62.102501 90.30625) (layer Edge.Cuts) (width 0.15))
   (gr_line (start 27.602501 70.80625) (end 62.102501 70.80625) (layer Edge.Cuts) (width 0.15))
   (gr_line (start 80.102501 51.80625) (end 80.102501 52.80625) (layer Edge.Cuts) (width 0.15))
