File: pcb/ukiha.kicad_pcb (KiCad board)
At the start: 2 copper layers, 200 x 88 mm, 143 parts, among them J1 Conn_01x03, SW1 SW_Push, SW10 SW_Push, SW11 SW_Push, SW12 SW_Push, SW13 SW_Push, SW14 SW_Push, SW15 SW_Push, SW16 SW_Push, SW17 SW_Push, SW18 SW_Push, SW19 SW_Push, SW2 SW_Push, SW20 SW_Push, SW21 SW_Push, SW22 SW_Push, SW23 SW_Push, SW24 SW_Push, SW25 SW_Push, SW26 SW_Push, SW27 SW_Push, SW28 SW_Push, SW29 SW_Push, SW3 SW_Push, SW30 SW_Push, SW31 SW_Push, SW32 SW_Push, SW33 SW_Push, SW34 SW_Push, SW35 SW_Push, SW36 SW_Push, SW37 SW_Push, SW38 SW_Push, SW39 SW_Push, SW4 SW_Push, SW40 SW_Push, SW41 SW_Push, SW42 SW_Push, SW43 SW_Push, SW44 SW_Push, SW45 SW_Push, SW46 SW_Push, SW47 SW_Push, SW48 SW_Push, SW49 SW_Push, SW5 SW_Push, SW50 SW_Push, SW51 SW_Push, SW52 SW_Push, SW53 SW_Push, SW54 SW_Push, SW55 SW_Push, SW56 SW_Push, SW57 SW_Push, SW58 SW_Push, SW59 SW_Push, SW6 SW_Push, SW60 SW_Push, SW61 SW_Push, SW62 SW_Push, SW63 SW_Push, SW7 SW_Push, SW8 SW_Push, SW9 SW_Push, U1 ProMicro/BLEMicroPro

Commit message: Add 48 key middle plate
Routing:
- net X12: track 227.0 -> 229.9 mm, vias 1 -> 0
Changed lines of the file:
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@@
     (pad_to_mask_clearance 0.2)
     (solder_mask_min_width 0.25)
-    (aux_axis_origin 37.70322 52.784508)
+    (aux_axis_origin 27.102501 36.80625)
     (grid_origin 27.102501 36.80625)
     (visible_elements 7FFFFFEF)
@@
   (segment (start 207.102501 56.80625) (end 207.102501 50.05625) (width 0.25) (layer B.Cu) (net 20))
   (segment (start 207.102501 57.20626) (end 207.102501 56.80625) (width 0.25) (layer B.Cu) (net 20))
-  (segment (start 210.7112 71.30625) (end 210.7112 71.30625) (width 0.25) (layer B.Cu) (net 20))
   (segment (start 211.292501 77.41625) (end 211.292501 78.26625) (width 0.25) (layer F.Cu) (net 20))
   (segment (start 211.767502 76.941249) (end 211.292501 77.41625) (width 0.25) (layer F.Cu) (net 20))
@@
   (segment (start 211.767502 65.365451) (end 211.767502 64.80625) (width 0.25) (layer F.Cu) (net 20))
   (segment (start 211.767502 71.30625) (end 211.767502 76.941249) (width 0.25) (layer F.Cu) (net 20))
-  (via (at 211.767502 71.30625) (size 0.8) (drill 0.4) (layers F.Cu B.Cu) (net 20))
-  (segment (start 69.117499 71.30625) (end 210.7112 71.30625) (width 0.25) (layer B.Cu) (net 20))
   (segment (start 68.602501 70.791252) (end 69.117499 71.30625) (width 0.25) (layer B.Cu) (net 20))
   (segment (start 58.852501 71.96625) (end 58.852501 70.30625) (width 0.25) (layer B.Cu) (net 20))
@@
   (segment (start 59.402491 69.75626) (end 67.552511 69.75626) (width 0.25) (layer B.Cu) (net 20))
   (segment (start 67.552511 69.75626) (end 68.587503 70.791252) (width 0.25) (layer B.Cu) (net 20))
-  (segment (start 210.7112 71.30625) (end 211.767502 71.30625) (width 0.25) (layer B.Cu) (net 20))
   (segment (start 68.587503 70.791252) (end 68.602501 70.791252) (width 0.25) (layer B.Cu) (net 20))
   (segment (start 211.292501 93.41625) (end 211.292501 94.26625) (width 0.25) (layer F.Cu) (net 20))
@@
   (segment (start 211.292501 79.11625) (end 211.767502 79.591251) (width 0.25) (layer F.Cu) (net 20))
   (segment (start 211.292501 78.26625) (end 211.292501 79.11625) (width 0.25) (layer F.Cu) (net 20))
+  (segment (start 205.182501 71.30625) (end 204.602501 71.30625) (width 0.25) (layer B.Cu) (net 20))
+  (segment (start 211.292501 77.41625) (end 205.182501 71.30625) (width 0.25) (layer B.Cu) (net 20))
+  (segment (start 211.292501 78.26625) (end 211.292501 77.41625) (width 0.25) (layer B.Cu) (net 20))
+  (segment (start 69.117499 71.30625) (end 204.602501 71.30625) (width 0.25) (layer B.Cu) (net 20))
   (segment (start 41.742501 42.87625) (end 41.742501 43.72625) (width 0.25) (layer B.Cu) (net 21))
   (segment (start 41.672501 42.80625) (end 41.742501 42.87625) (width 0.25) (layer B.Cu) (net 21))

Commit message: Fix PCB
Parts:
- removed D61, D62, D63: D, #footprint:diode_SMD
- SW53, SW54, SW55, SW56, SW57, SW58, SW59, SW60, SW61, SW62, SW63: footprint #footprint:CherryMX_MidHeight_16mm_rev3 -> #footprint:CherryMX_MidHeight_16mm_rev2
- moved J1 2.50 mm to (36.6, 105.5)
- moved ? 0.71 mm to (224.6, 106.3)
- moved ? 0.71 mm to (29.6, 106.3)
- moved ? 0.71 mm to (29.6, 122.3)
- moved ? 0.71 mm to (29.6, 55.3)
- moved ? 0.71 mm to (29.6, 39.3)
- moved ? 0.71 mm to (224.6, 39.3)
- moved ? 0.71 mm to (224.6, 55.3)
- moved ? 0.71 mm to (224.6, 122.3)
- moved ? 0.50 mm to (159.1, 55.3)
- moved ? 0.50 mm to (95.1, 55.3)
- moved ? 0.50 mm to (95.1, 122.3)
- moved ? 0.50 mm to (159.1, 122.3)
- moved ? 0.50 mm to (159.1, 39.3)
- moved ? 0.50 mm to (95.1, 39.3)
Connections:
- SW61 pad 2: Net-(D61-Pad2) -> Net-(D53-Pad2)
- SW62 pad 2: Net-(D62-Pad2) -> Net-(D55-Pad2)
- SW63 pad 2: Net-(D63-Pad2) -> Net-(D54-Pad2)
Routing:
- net Net-(D63-Pad2): track 67.2 -> 0.00 mm, vias 1 -> 0
- net Net-(D61-Pad2): track 41.0 -> 0.00 mm, vias 1 -> 0
- net Net-(D62-Pad2): track 31.2 -> 0.00 mm, vias 1 -> 0
- net Net-(D53-Pad2): track 22.5 -> 30.5 mm
- net Net-(D54-Pad2): track 58.8 -> 65.0 mm
- net VCC: track 35.4 -> 37.9 mm
- net GND: track 47.7 -> 50.2 mm
- net Y5: track 216.7 -> 214.8 mm
- net Net-(D55-Pad2): track 49.3 -> 50.8 mm
- net led: track 18.4 -> 17.8 mm
Other:
- net class Default: trace_width 0.25 -> 0.5
